File: accelerometer-daughterboard.sch (EAGLE design)
At the start: 4 parts, among them U1 LIS3DHTR

Commit message: Complete first board draft, including outline and wiring
Connections:
- net GND: now also U1.NC@1, U1.NC@2
Changed lines of the file:
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@@
 <part name="R34" library="rcl" library_urn="urn:adsk.eagle:library:334" deviceset="R-EU_" device="R0603" package3d_urn="urn:adsk.eagle:package:23555/3" value="10K"/>
 <part name="U$3" library="microbuilder" deviceset="GND" device=""/>
+<part name="U$5" library="microbuilder" deviceset="GND" device=""/>
 </parts>
 <sheets>
@@
 <attribute name="VALUE" x="110.236" y="101.6" size="1.27" layer="96"/>
 </instance>
+<instance part="U$5" gate="G$1" x="66.04" y="53.34" smashed="yes">
+<attribute name="VALUE" x="64.516" y="50.8" size="1.27" layer="96"/>
+</instance>
 </instances>
 <busses>
@@
 <wire x1="111.76" y1="106.68" x2="111.76" y2="109.22" width="0.1524" layer="91"/>
 </segment>
+<segment>
+<pinref part="U$5" gate="G$1" pin="GND"/>
+<wire x1="66.04" y1="55.88" x2="66.04" y2="66.04" width="0.1524" layer="91"/>
+<pinref part="U1" gate="G$1" pin="NC@1"/>
+<wire x1="88.9" y1="66.04" x2="86.36" y2="66.04" width="0.1524" layer="91"/>
+<wire x1="86.36" y1="66.04" x2="86.36" y2="63.5" width="0.1524" layer="91"/>
+<pinref part="U1" gate="G$1" pin="NC@2"/>
+<wire x1="86.36" y1="63.5" x2="88.9" y2="63.5" width="0.1524" layer="91"/>
+<wire x1="66.04" y1="66.04" x2="86.36" y2="66.04" width="0.1524" layer="91"/>
+<junction x="86.36" y="66.04"/>
+</segment>
 </net>

Commit message: Rename SD0 to SA0; add measures
Connections:
- net SDO renamed SAO
Changed lines of the file:
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@@
 </segment>
 </net>
-<net name="SDO" class="0">
+<net name="SAO" class="0">
 <segment>
 <pinref part="U1" gate="G$1" pin="SDO"/>

Commit message: Tweak
Connections:
- net INT1: now also U$1.4
- net SAO: no longer U$1.4
Changed lines of the file:
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@@
 <label x="121.92" y="63.5" size="1.778" layer="95"/>
+</segment>
+<segment>
+<pinref part="U$1" gate="G$1" pin="4"/>
+<wire x1="104.14" y1="109.22" x2="104.14" y2="96.52" width="0.1524" layer="91"/>
+<label x="104.14" y="96.52" size="1.778" layer="95" rot="R90"/>
 </segment>
 </net>
@@
 <label x="104.14" y="33.02" size="1.778" layer="95" rot="R90"/>
 </segment>
-<segment>
-<pinref part="U$1" gate="G$1" pin="4"/>
-<wire x1="104.14" y1="109.22" x2="104.14" y2="96.52" width="0.1524" layer="91"/>
-<label x="104.14" y="96.52" size="1.778" layer="95" rot="R90"/>
-</segment>
 </net>

Commit message: Re-add buffer caps
Parts:
- added C1: 0.1uF, microbuilder:CAP_CERAMIC0603_NO
- added C3: 10uF, microbuilder:CAP_CERAMIC0805-NOOUTLINE
Changed lines of the file:
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@@
 </classes>
 <parts>
+<part name="C3" library="microbuilder" deviceset="CAP_CERAMIC" device="0805-NOOUTLINE" value="10uF"/>
+<part name="C1" library="microbuilder" deviceset="CAP_CERAMIC" device="0603_NO" value="0.1uF"/>
 <part name="U$7" library="microbuilder" deviceset="3.3V" device=""/>
 <part name="U$24" library="microbuilder" deviceset="3.3V" device=""/>
@@
 <attribute name="SHEET" x="230.505" y="10.16" size="2.54" layer="94" font="vector"/>
 </instance>
+<instance part="C3" gate="G$1" x="50.8" y="154.94" smashed="yes">
+<attribute name="NAME" x="48.51" y="156.19" size="1.27" layer="95" font="vector" rot="R90" align="center"/>
+<attribute name="VALUE" x="53.1" y="156.19" size="1.27" layer="96" font="vector" rot="R90" align="center"/>
+</instance>
+<instance part="C1" gate="G$1" x="60.96" y="154.94" smashed="yes">
+<attribute name="NAME" x="58.67" y="156.19" size="1.27" layer="95" font="vector" rot="R90" align="center"/>
+<attribute name="VALUE" x="63.26" y="156.19" size="1.27" layer="96" font="vector" rot="R90" align="center"/>
+</instance>
 <instance part="U$7" gate="G$1" x="165.1" y="170.18" smashed="yes" rot="MR0">

Commit message: remove caps again
Parts:
- removed C1: 0.1uF, microbuilder:CAP_CERAMIC0603_NO
- removed C3: 10uF, microbuilder:CAP_CERAMIC0805-NOOUTLINE
Changed lines of the file:
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@@
 </classes>
 <parts>
-<part name="C3" library="microbuilder" deviceset="CAP_CERAMIC" device="0805-NOOUTLINE" value="10uF"/>
-<part name="C1" library="microbuilder" deviceset="CAP_CERAMIC" device="0603_NO" value="0.1uF"/>
 <part name="U$7" library="microbuilder" deviceset="3.3V" device=""/>
 <part name="U$24" library="microbuilder" deviceset="3.3V" device=""/>
@@
 <attribute name="SHEET" x="230.505" y="10.16" size="2.54" layer="94" font="vector"/>
 </instance>
-<instance part="C3" gate="G$1" x="50.8" y="154.94" smashed="yes">
-<attribute name="NAME" x="48.51" y="156.19" size="1.27" layer="95" font="vector" rot="R90" align="center"/>
-<attribute name="VALUE" x="53.1" y="156.19" size="1.27" layer="96" font="vector" rot="R90" align="center"/>
-</instance>
-<instance part="C1" gate="G$1" x="60.96" y="154.94" smashed="yes">
-<attribute name="NAME" x="58.67" y="156.19" size="1.27" layer="95" font="vector" rot="R90" align="center"/>
-<attribute name="VALUE" x="63.26" y="156.19" size="1.27" layer="96" font="vector" rot="R90" align="center"/>
-</instance>
 <instance part="U$7" gate="G$1" x="165.1" y="170.18" smashed="yes" rot="MR0">
